Commit message: move robot with turtletele

File: src/my_r2d2/urdf/r2d2_ex4.urdf.xacro (robot description, xacro)
@@ -37,4 +37,12 @@
     <xacro:default_inertial mass="10"/>
   </link>
+  <link name="base_footprint">
+  <origin xyz="0 0 0"/>
+  </link>
+  <joint name="base_footprint_to_base_link" type="fixed">
+    <parent link="base_footprint"/>
+    <child link="base_link"/>
+    <origin xyz="0 0 ${(baselen + wheeldiam/2)} "/>
+  </joint>
   <xacro:macro name="wheel" params="prefix suffix reflect">
     <link name="${prefix}_${suffix}_wheel">

Commit message: pooleli

File: src/my_r2d2/urdf/r2d2_ex4.urdf.xacro (robot description, xacro)
@@ -221,5 +221,5 @@
     <origin xyz="${.707*width+0.04} 0 ${.707*width}"/>
   </joint>
-  <link name="lens">
+  <link name="lense">
     <visual>
       <geometry>
@@ -236,7 +236,15 @@
     <xacro:default_inertial mass="1"/>
   </link>
-  <joint name="tolens" type="fixed">
+  <link name="eye">
+      <origin xyz="0 0 0" rpy="0 ${pi/2} 0"/>
+  </link>
+  <joint name="toeye" type="fixed">
+    <parent link="lense"/>
+    <child link="eye"/>
+    <origin rpy="0 ${pi/2} 0" />
+  </joint>
+  <joint name="tolense" type="fixed">
     <parent link="box"/>
-    <child link="lens"/>
+    <child link="lense"/>
     <origin xyz="0 0 0"/>
   </joint>
